File: for-science.kicad_pcb (KiCad board)
At the start: 2 copper layers, 92 x 92 mm, 57 parts, among them J1 TRRS, J2 TRRS, M8 MountingHole_8.4mm_M8, U1 ARDUINO_PRO_MICRO

Commit message: initial attempts
Parts:
- removed D27, D28: DIODE, keyboard_parts:D_SOD123_axial
- removed GROUND1: Ground, keyboard_parts:PIN_1_SQUARE
- removed J1: TRRS, Keyboard:PJ320D_3.5mm_Jack_SMD
- removed J2: TRRS, Keyboard:PJ320D_3.5mm_Jack_SMD_Flip
- removed MX4:3: MX4:6, Keyboard:MX_DoubleSided
- removed MX4:4: MX4:5, Keyboard:MX_DoubleSided
- removed RESET1: Reset, keyboard_parts:PIN_1_SQUARE
- added J*: MJ-4PP-9, kbd:MJ-4PP-9, F.Cu at (11.6, -1.15)
- D1, D10, D11, D13, D14, D15, D16, D17, D19, D2, D20, D21, D22, D23, D26, D3, D4, D5, D7, D8, D9: footprint keyboard_parts:D_SOD123_axial -> kbd:D3_TH_SMD_v2
- MX0:0, MX0:1, MX0:2, MX0:3, MX0:4, MX1:0, MX1:1, MX1:2, MX1:3, MX1:4, MX2:0, MX2:1, MX2:2, MX2:3, MX2:4, MX3:0, MX3:1, MX3:2, MX3:3, MX3:4, MX4:2: footprint Keyboard:MX_DoubleSided -> keyswitches:SW_PG1350_reversible_nohole
- U1: value ARDUINO_PRO_MICRO -> ProMicro; footprint footprints:ARDUINO_PRO_MICRO -> kbd:ProMicro_v2
- moved EXTRADATA1 171.2 mm to (7.75, -4.00), turned to 90 degrees
- moved M8 169.0 mm to (320.5, 84.0)
- moved M8 169.0 mm to (320.5, 27.0)
- moved M8 169.0 mm to (263.5, 27.0)
- moved M8 169.0 mm to (263.5, 65.0)
- moved TX0 143.1 mm to (-5.75, 9.75)
- moved U1 120.2 mm to (11.2, 31.5), turned to 0 degrees
- moved MX3:0 109.5 mm to (182.5, 54.0), turned to 180 degrees
- moved D19 98.9 mm to (182.5, 58.8), turned to 0 degrees
- moved MX3:1 84.3 mm to (182.5, 71.5), turned to 180 degrees
- moved D20 73.7 mm to (182.5, 76.2), turned to 0 degrees
- moved MX4:2 69.0 mm to (182.5, 89.0), turned to 180 degrees
- moved D26 58.5 mm to (182.5, 93.8), turned to 0 degrees
- moved MX3:2 55.7 mm to (182.5, 106.5), turned to 180 degrees
- moved D21 46.0 mm to (182.5, 111.2), turned to 0 degrees
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Routing:
- net /Col4: track 137.9 -> 14.4 mm
- net /Row2: track 118.6 -> 17.1 mm
- net /Row3: track 115.0 -> 17.1 mm
- net GND: track 110.5 -> 17.1 mm, vias 1 -> 0
- net /Col0: track 107.4 -> 14.4 mm
- net /Row4: track 106.5 -> 17.1 mm
- net /Row1: track 106.1 -> 17.1 mm
- net /Col3: track 100.5 -> 14.4 mm
- net /Col1: track 88.3 -> 14.4 mm
- net /Col2: track 87.2 -> 14.4 mm
- net /Row0: track 89.7 -> 17.1 mm
- net Net-(J1-Pad1): track 62.5 -> 17.1 mm, vias 1 -> 0
- net Net-(EXTRADATA1-Pad1): track 43.1 -> 0.00 mm, vias 1 -> 0
- net VCC: track 57.5 -> 14.4 mm, vias 1 -> 0
- net Net-(D3-Pad1): track 37.8 -> 0.00 mm
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Other:
- board outline removed
- net class Default removed
- board text removed: "Chip side down"
- board text removed: "Chip side up"
- board text removed: "Left hand"
- board text removed: "Pro Micro"
- board text removed: "Right hand"
